Commit message: Change base link and base footprint frames hierarchy

File: sml_nexus_description/urdf/sml_nexus.xacro (robot description, xacro)
@@ -8,34 +8,34 @@
   <material name="dark_grey"><color rgba="0.2 0.2 0.2 1.0" /></material>
   <material name="light_grey"><color rgba="0.4 0.4 0.4 1.0" /></material>
+  <link name="base_link">
+    <visual>
+      <origin xyz="0 0 0" rpy="0 0 ${PI}" />
+      <geometry>
+        <mesh filename="package://sml_nexus_description/meshes/nexus_base_link.STL" scale="0.001 0.001 0.001"/>
+      </geometry>
+      <material name="yellow" />
+    </visual>
+    <collision>
+      <origin xyz="0 0 ${PI}"/>
+      <geometry>
+        <mesh filename="package://sml_nexus_description/meshes/nexus_base_link_collision.STL" scale="0.001 0.001 0.001"/>
+      </geometry>
+    </collision>
+    <inertial>
+      <!-- Inertia from CAD model, filled box assumption -->
+      <origin xyz="0.01103 0 0.002" rpy="0 0 ${PI}"/>
+      <mass value="2.844"/>
+      <inertia
+        ixx="0.018819942" ixy="0" ixz="-0.000101519"
+        iyy="0.057333716" iyz="0"
+        izz="0.074201740"/>
+    </inertial>
+  </link>
   <link name="base_footprint"></link>
   <joint name="base_link_joint" type="fixed">
     <origin xyz="0 0 0.05" rpy="0 0 0" />
-    <parent link="base_footprint"/>
-    <child link="base_link" />
-  </joint>
-  <link name="base_link">
-    <visual>
-      <origin xyz="0 0 0" rpy="0 0 ${PI}" />
-      <geometry>
-        <mesh filename="package://sml_nexus_description/meshes/nexus_base_link.STL" scale="0.001 0.001 0.001"/>
-      </geometry>
-      <material name="yellow" />
-    </visual>
-    <collision>
-      <origin xyz="0 0 ${PI}"/>
-      <geometry>
-        <mesh filename="package://sml_nexus_description/meshes/nexus_base_link_collision.STL" scale="0.001 0.001 0.001"/>
-      </geometry>
-    </collision>
-    <inertial>
-      <!-- Inertia from CAD model, filled box assumption -->
-      <origin xyz="0.01103 0 0.002" rpy="0 0 ${PI}"/>
-      <mass value="2.844"/>
-      <inertia
-        ixx="0.018819942" ixy="0" ixz="-0.000101519"
-        iyy="0.057333716" iyz="0"
-        izz="0.074201740"/>
-    </inertial>
-  </link>
+    <parent link="base_link"/>
+    <child link="base_footprint" />
+  </joint>
   <joint name="upper_left_wheel_shaft_joint" type="fixed">
     <origin xyz="0.150 0.108 0.0" rpy="0 0 0" />

Commit message: Fix URDF with replacing root link with dummy one

File: sml_nexus_description/urdf/sml_nexus.xacro (robot description, xacro)
@@ -8,5 +8,7 @@
   <material name="dark_grey"><color rgba="0.2 0.2 0.2 1.0" /></material>
   <material name="light_grey"><color rgba="0.4 0.4 0.4 1.0" /></material>
-  <link name="base_link">
+  <link name="base_link"></link>
+  <link name="base_footprint"></link>
+  <link name="nexus_body">
     <visual>
       <origin xyz="0 0 0" rpy="0 0 ${PI}" />
@@ -32,13 +34,17 @@
     </inertial>
   </link>
-  <link name="base_footprint"></link>
   <joint name="base_link_joint" type="fixed">
+    <origin xyz="0 0 0" rpy="0 0 0" />
+    <parent link="base_link"/>
+    <child link="base_footprint" />
+  </joint>
+  <joint name="nexus_body_joint" type="fixed">
     <origin xyz="0 0 0.05" rpy="0 0 0" />
     <parent link="base_link"/>
-    <child link="base_footprint" />
+    <child link="nexus_body" />
   </joint>
   <joint name="upper_left_wheel_shaft_joint" type="fixed">
     <origin xyz="0.150 0.108 0.0" rpy="0 0 0" />
-    <parent link="base_link"/>
+    <parent link="nexus_body"/>
     <child link="upper_left_wheel_shaft" />
   </joint>
@@ -68,5 +74,5 @@
   <joint name="lower_left_wheel_shaft_joint" type="fixed">
     <origin xyz="-0.150 0.108 0.0" rpy="0 0 0" />
-    <parent link="base_link"/>
+    <parent link="nexus_body"/>
     <child link="lower_left_wheel_shaft" />
   </joint>
@@ -96,5 +102,5 @@
   <joint name="upper_right_wheel_shaft_joint" type="fixed">
     <origin xyz="0.150 -0.108 0.0" rpy="${PI} 0 0" />
-    <parent link="base_link"/>
+    <parent link="nexus_body"/>
     <child link="upper_right_wheel_shaft" />
   </joint>
@@ -124,5 +130,5 @@
   <joint name="lower_right_wheel_shaft_joint" type="fixed">
     <origin xyz="-0.150 -0.108 0.0" rpy="${PI} 0 0" />
-    <parent link="base_link"/>
+    <parent link="nexus_body"/>
     <child link="lower_right_wheel_shaft" />
   </joint>
@@ -272,5 +278,5 @@
   <joint name="left_sensor_joint" type="fixed">
     <origin xyz="0 0.108 0.010" rpy="0 0 ${PI/2}" />
-    <parent link="base_link"/>
+    <parent link="nexus_body"/>
     <child link="left_sensor" />
   </joint>
@@ -286,5 +292,5 @@
   <joint name="front_sensor_joint" type="fixed">
     <origin xyz="0.201 0 0.010" rpy="0 0 0" />
-    <parent link="base_link"/>
+    <parent link="nexus_body"/>
     <child link="front_sensor" />
   </joint>
@@ -300,5 +306,5 @@
   <joint name="right_sensor_joint" type="fixed">
     <origin xyz="0 -0.108 0.010" rpy="0 0 ${-PI/2}" />
-    <parent link="base_link"/>
+    <parent link="nexus_body"/>
     <child link="right_sensor" />
   </joint>
@@ -314,5 +320,5 @@
   <joint name="rear_sensor_joint" type="fixed">
     <origin xyz="-0.205 0 0.010" rpy="0 0 ${PI}" />
-    <parent link="base_link"/>
+    <parent link="nexus_body"/>
     <child link="rear_sensor" />
   </joint>
